File: hardware/schematics/Breeze.kicad_sch (KiCad schematic)
At the start: 7 parts, among them U1 WEMOS_D1_mini, U3 BME280

Commit message: Schematic added
KiCAD and PDF schematic added
Parts:
- removed R2: 10k, symbol Device:R
Connections:
- net at U2.6 (RST): now also U1.5 (MISO/D6); no longer U1.3 (D0)
- net at U2.4 (RXD): now also U1.7 (CS/D8); no longer U1.6 (MOSI/D7)
- net at U2.5 (TXD): now also U1.6 (MOSI/D7); no longer U1.5 (MISO/D6)
Other:
- title: (none) -> Breeze Indoor Air Quality Monitor – Schematic
Changed lines of the file:
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@@
 	(generator_version "9.0")
 	(paper "A4")
+	(title_block
+		(title "Breeze Indoor Air Quality Monitor – Schematic")
+		(date "2026-03-05")
+		(rev "00alpha")
+	)
 	(junction
 		(at 177.8 67.31)
@@
 	)
 	(junction
-		(at 121.92 83.82)
-		(diameter 0)
-		(color 0 0 0 0)
-	)
-	(junction
 		(at 143.51 118.11)
 		(diameter 0)
@@
 	)
 	(junction
-		(at 121.92 67.31)
-		(diameter 0)
-		(color 0 0 0 0)
-	)
-	(junction
 		(at 158.75 120.65)
 		(diameter 0)
@@
 	(wire
 		(pts
+			(xy 167.64 125.73) (xy 167.64 104.14)
+		)
+		(stroke
+			(width 0)
+			(type default)
+		)
+	)
+	(wire
+		(pts
 			(xy 158.75 88.9) (xy 115.57 88.9)
 		)
@@
 	(wire
 		(pts
+			(xy 165.1 128.27) (xy 165.1 101.6)
+		)
+		(stroke
+			(width 0)
+			(type default)
+		)
+	)
+	(wire
+		(pts
 			(xy 172.72 128.27) (xy 165.1 128.27)
 		)
@@
 	(wire
 		(pts
-			(xy 167.64 101.6) (xy 115.57 101.6)
-		)
-		(stroke
-			(width 0)
-			(type default)
-		)
-	)
-	(wire
-		(pts
 			(xy 201.93 67.31) (xy 177.8 67.31)
 		)
@@
 	(wire
 		(pts
-			(xy 127 130.81) (xy 127 83.82)
+			(xy 165.1 101.6) (xy 115.57 101.6)
 		)
 		(stroke
@@
 	(wire
 		(pts
-			(xy 167.64 125.73) (xy 167.64 101.6)
-		)
-		(stroke
-			(width 0)
-			(type default)
-		)
-	)
-	(wire
-		(pts
-			(xy 121.92 67.31) (xy 121.92 71.12)
-		)
-		(stroke
-			(width 0)
-			(type default)
-		)
-	)
-	(wire
-		(pts
 			(xy 102.87 63.5) (xy 102.87 73.66)
 		)
@@
 	(wire
 		(pts
-			(xy 127 83.82) (xy 121.92 83.82)
-		)
-		(stroke
-			(width 0)
-			(type default)
-		)
-	)
-	(wire
-		(pts
 			(xy 158.75 120.65) (xy 133.35 120.65)
 		)
@@
 	(wire
 		(pts
+			(xy 127 99.06) (xy 115.57 99.06)
+		)
+		(stroke
+			(width 0)
+			(type default)
+		)
+	)
+	(wire
+		(pts
 			(xy 102.87 59.69) (xy 102.87 63.5)
 		)
@@
 	(wire
 		(pts
-			(xy 121.92 67.31) (xy 138.43 67.31)
+			(xy 107.95 67.31) (xy 138.43 67.31)
+		)
+		(stroke
+			(width 0)
+			(type default)
+		)
+	)
+	(wire
+		(pts
+			(xy 127 130.81) (xy 127 99.06)
 		)
 		(stroke
@@
 	(wire
 		(pts
-			(xy 165.1 128.27) (xy 165.1 99.06)
-		)
-		(stroke
-			(width 0)
-			(type default)
-		)
-	)
-	(wire
-		(pts
 			(xy 172.72 123.19) (xy 170.18 123.19)
 		)
@@
 	(wire
 		(pts
-			(xy 107.95 67.31) (xy 121.92 67.31)
-		)
-		(stroke
-			(width 0)
-			(type default)
-		)
-	)
-	(wire
-		(pts
 			(xy 201.93 78.74) (xy 201.93 67.31)
 		)
@@
 	(wire
 		(pts
-			(xy 121.92 83.82) (xy 115.57 83.82)
-		)
-		(stroke
-			(width 0)
-			(type default)
-		)
-	)
-	(wire
-		(pts
 			(xy 115.57 86.36) (xy 161.29 86.36)
 		)
@@
 	(wire
 		(pts
+			(xy 167.64 104.14) (xy 115.57 104.14)
+		)
+		(stroke
+			(width 0)
+			(type default)
+		)
+	)
+	(wire
+		(pts
 			(xy 129.54 118.11) (xy 143.51 118.11)
 		)
@@
 	(wire
 		(pts
-			(xy 121.92 78.74) (xy 121.92 83.82)
-		)
-		(stroke
-			(width 0)
-			(type default)
-		)
-	)
-	(wire
-		(pts
 			(xy 143.51 113.03) (xy 143.51 118.11)
 		)
@@
 		(pts
 			(xy 201.93 99.06) (xy 177.8 99.06)
-		)
-		(stroke
-			(width 0)
-			(type default)
-		)
-	)
-	(wire
-		(pts
-			(xy 165.1 99.06) (xy 115.57 99.06)
 		)
 		(stroke
@@
 					(unit 1)
 				)
-			)
-		)
-	)
-	(symbol
-		(lib_id "Device:R")
-		(at 121.92 74.93 0)
-		(unit 1)
-		(exclude_from_sim no)
-		(in_bom yes)
-		(on_board yes)
-		(dnp no)
-		(fields_autoplaced yes)
-		(property "Reference" "R2"
-			(at 124.46 73.6599 0)
-			(effects
-				(font
-					(size 1.27 1.27)
-				)
-				(justify left)
-			)
-		)
-		(property "Value" "10k"
-			(at 124.46 76.1999 0)
-			(effects
-				(font
-					(size 1.27 1.27)
-				)
-				(justify left)
-			)
-		)
-		(property "Footprint" ""
-			(at 120.142 74.93 90)
-			(effects
-				(font
-					(size 1.27 1.27)
-				)
-				(hide yes)
-			)
-		)
-		(property "Datasheet" "~"
-			(at 121.92 74.93 0)
-			(effects
-				(font
-					(size 1.27 1.27)
-				)
-				(hide yes)
-			)
-		)
-		(property "Description" "Resistor"
-			(at 121.92 74.93 0)
-			(effects
-				(font
-					(size 1.27 1.27)
-				)
-				(hide yes)
-			)
-		)
-		(pin "1"
-		)
-		(pin "2"
-		)
-		(instances
-			(project "Breeze"
-				(path "/f1965451-c1dc-41a0-abe4-45483b23ddd7"
-					(reference "R2")
-					(unit 1)
-				)
